File: Design/Projector/DLP_Board/dlp_01/dlp_01_sch_brd/dlp_controller_config.sch (KiCad schematic (older format))
At the start: 46 parts

Commit message: Updated schematic with changes pulling together top level design
Connections:
- net at U?.P11 (RESERVED8): now also R?.2 (x2)
Changed lines of the file:
@@
 EESchema Schematic File Version 4
+LIBS:dlp_01-cache
 EELAYER 29 0
 EELAYER END

Commit message: More updates in the DLP board
Parts:
- added R? (x8): 0R, Resistors_SMD:R_0603, symbol Device:R
Connections:
- net at U?.P11 (RESERVED8): now also R?.2 (x2)
- net mI2C_SCL: no longer names the net of R?.2, U?.R11 (IIC1_SCL)
- net mI2C_SCL: now also R?.1; no longer U?.N10 (IIC0_SCL)
- net mI2C_SDA: no longer names the net of R?.2, U?.R10 (IIC1_SDA)
- net mI2C_SDA: now also R?.2; no longer U?.N9 (IIC0_SDA)
- net sI2C_SCL: no longer names the net of R?.2, U?.R11 (IIC1_SCL)
- net sI2C_SCL: now also R?.1; no longer U?.N10 (IIC0_SCL)
- net sI2C_SDA: no longer names the net of R?.2, U?.R10 (IIC1_SDA)
- net sI2C_SDA: now also R?.2; no longer U?.N9 (IIC0_SDA)
- new net: R?.1, U?.N10 (IIC0_SCL) (x2)
- new net: R?.2, U?.N9 (IIC0_SDA) (x2)
- new net mI2C0_SCL: R?.2
- new net mI2C0_SDA: R?.1
- new net mI2C1_SCL: R?.2
- new net mI2C1_SDA: R?.1
- new net sI2C0_SCL: R?.2
- new net sI2C0_SDA: R?.1
- new net sI2C1_SCL: R?.2
- new net sI2C1_SDA: R?.1
Changed lines of the file:
@@
 Wire Wire Line
 	4300 2250 4300 2150
-Text HLabel 5900 3750 0    50   Output ~ 0
-mI2C_SCL
-Text HLabel 5900 3850 0    50   BiDi ~ 0
-mI2C_SDA
+Text HLabel 5400 3750 0    50   Output ~ 0
+mI2C0_SCL
+Text HLabel 5400 3850 0    50   BiDi ~ 0
+mI2C0_SDA
 Wire Wire Line
 	5900 3850 6100 3850
@@
 Wire Wire Line
 	4850 3900 4850 4000
-Text HLabel 3350 4350 0    50   Output ~ 0
-mI2C_SCL
-Text HLabel 3350 4450 0    50   BiDi ~ 0
-mI2C_SDA
+Text HLabel 2900 4350 0    50   Output ~ 0
+mI2C1_SCL
+Text HLabel 2900 4450 0    50   BiDi ~ 0
+mI2C1_SDA
 $Comp
 L Memory_Flash:W25Q32JVSS U?
@@
 Wire Wire Line
 	11950 2250 11950 2150
-Text HLabel 13550 3750 0    50   Output ~ 0
-sI2C_SCL
-Text HLabel 13550 3850 0    50   BiDi ~ 0
-sI2C_SDA
-Wire Wire Line
-	13550 3850 13750 3850
-Wire Wire Line
-	13550 3750 13750 3750
+Text HLabel 13050 3750 0    50   Output ~ 0
+sI2C0_SCL
+Text HLabel 13050 3850 0    50   BiDi ~ 0
+sI2C0_SDA
+Wire Wire Line
+	13050 3850 13250 3850
+Wire Wire Line
+	13050 3750 13250 3750
 $Comp
 L Device:R R?
@@
 Wire Wire Line
 	12500 3900 12500 4000
-Text HLabel 11050 4350 0    50   Output ~ 0
-sI2C_SCL
-Text HLabel 11050 4450 0    50   BiDi ~ 0
-sI2C_SDA
+Text HLabel 10650 4350 0    50   Output ~ 0
+sI2C1_SCL
+Text HLabel 10650 4450 0    50   BiDi ~ 0
+sI2C1_SDA
 Wire Wire Line
 	13350 5300 13750 5300
@@
 	11050 4450 11900 4450
 Connection ~ 11900 4450
-Text HLabel 11050 4650 0    50   Output ~ 0
+Text HLabel 11050 4950 0    50   Output ~ 0
 sHOST_IRQ
 Wire Wire Line
-	11050 4650 11300 4650
-Wire Wire Line
 	11300 4300 11300 4650
-Connection ~ 11300 4650
 Wire Wire Line
 	11300 4650 13750 4650
@@
 	1    0    0    -1
 $EndComp
-Text HLabel 3350 4650 0    50   Output ~ 0
+Text HLabel 3450 4950 0    50   Output ~ 0
 mHOST_IRQ
-Wire Wire Line
-	3350 4650 3650 4650
 Wire Wire Line
 	3350 4350 4850 4350
@@
 Wire Wire Line
 	8500 7250 8750 7250
+$Comp
+L Device:R R?
+U 1 1 5E9414B5
+P 13400 3750
+F 0 "R?" V 13141 3750 50  0000 C CNN
+F 1 "0R" V 13232 3750 50  0000 C CNN
+F 2 "Resistors_SMD:R_0603" V 13304 3750 25  0000 C CNN
+F 3 "~" H 13400 3750 50  0001 C CNN
+	1    13400 3750
+	0    1    1    0
+$EndComp
+$Comp
+L Device:R R?
+U 1 1 5E941DED
+P 13400 3850
+F 0 "R?" V 13141 3850 50  0000 C CNN
+F 1 "0R" V 13232 3850 50  0000 C CNN
+F 2 "Resistors_SMD:R_0603" V 13304 3850 25  0000 C CNN
+F 3 "~" H 13400 3850 50  0001 C CNN
+	1    13400 3850
+	0    -1   -1   0
+$EndComp
+Wire Wire Line
+	13550 3750 13750 3750
+Wire Wire Line
+	13550 3850 13750 3850
+$Comp
+L Device:R R?
+U 1 1 5E962D93
+P 10900 4350
+F 0 "R?" V 10641 4350 50  0000 C CNN
+F 1 "0R" V 10732 4350 50  0000 C CNN
+F 2 "Resistors_SMD:R_0603" V 10804 4350 25  0000 C CNN
+F 3 "~" H 10900 4350 50  0001 C CNN
+	1    10900 4350
+	0    1    1    0
+$EndComp
+$Comp
+L Device:R R?
+U 1 1 5E962D9D
+P 10900 4450
+F 0 "R?" V 10641 4450 50  0000 C CNN
+F 1 "0R" V 10732 4450 50  0000 C CNN
+F 2 "Resistors_SMD:R_0603" V 10804 4450 25  0000 C CNN
+F 3 "~" H 10900 4450 50  0001 C CNN
+	1    10900 4450
+	0    -1   -1   0
+$EndComp
+Wire Wire Line
+	11050 4950 11300 4950
+Wire Wire Line
+	11300 4950 11300 4650
+Connection ~ 11300 4650
+Wire Wire Line
+	10650 4350 10750 4350
+Wire Wire Line
+	10750 4450 10650 4450
+$Comp
+L Device:R R?
+U 1 1 5E9CD6E4
+P 5750 3750
+F 0 "R?" V 5491 3750 50  0000 C CNN
+F 1 "0R" V 5582 3750 50  0000 C CNN
+F 2 "Resistors_SMD:R_0603" V 5654 3750 25  0000 C CNN
+F 3 "~" H 5750 3750 50  0001 C CNN
+	1    5750 3750
+	0    1    1    0
+$EndComp
+$Comp
+L Device:R R?
+U 1 1 5E9CD6EE
+P 5750 3850
+F 0 "R?" V 5491 3850 50  0000 C CNN
+F 1 "0R" V 5582 3850 50  0000 C CNN
+F 2 "Resistors_SMD:R_0603" V 5654 3850 25  0000 C CNN
+F 3 "~" H 5750 3850 50  0001 C CNN
+	1    5750 3850
+	0    -1   -1   0
+$EndComp
+Wire Wire Line
+	5400 3850 5600 3850
+Wire Wire Line
+	5400 3750 5600 3750
+$Comp
+L Device:R R?
+U 1 1 5EA29549
+P 3200 4350
+F 0 "R?" V 2941 4350 50  0000 C CNN
+F 1 "0R" V 3032 4350 50  0000 C CNN
+F 2 "Resistors_SMD:R_0603" V 3104 4350 25  0000 C CNN
+F 3 "~" H 3200 4350 50  0001 C CNN
+	1    3200 4350
+	0    1    1    0
+$EndComp
+$Comp
+L Device:R R?
+U 1 1 5EA29553
+P 3200 4450
+F 0 "R?" V 2941 4450 50  0000 C CNN
+F 1 "0R" V 3032 4450 50  0000 C CNN
+F 2 "Resistors_SMD:R_0603" V 3104 4450 25  0000 C CNN
+F 3 "~" H 3200 4450 50  0001 C CNN
+	1    3200 4450
+	0    -1   -1   0
+$EndComp
+Wire Wire Line
+	3450 4950 3650 4950
+Wire Wire Line
+	3650 4950 3650 4650
+Wire Wire Line
+	2900 4350 3050 4350
+Wire Wire Line
+	3050 4450 2900 4450
 $EndSCHEMATC

Commit message: Initial placement of power converters, BGA fanout and Z-turn board outline imported
Parts:
- added C100, C99: 100n, Capacitors_SMD:C_0603, symbol Device:C
- added TP10: TestPoint, Measurement_Points:Measurement_Point_Round-SMD-Pad_Small, symbol Connector:TestPoint
- U3: renamed from U?; footprint Oscillator:Oscillator_SMD_Abracon_ASDMB-4Pin_2.5x2.0mm -> Oscillators:Oscillator_SMD_SeikoEpson_SG210-4pin_2.5x2.0mm_HandSoldering
- U4, U5: renamed from U?; footprint Package_SO:SOIC-8_5.23x5.23mm_P1.27mm -> Housings_SOIC:SO-8_5.3x6.2mm_Pitch1.27mm
- gave numbers to parts that had none: 45
Connections:
- net +3V3: now also C100.1, C99.1
- net GND: now also C100.2, C99.2
- net at U1.A15 (CMP_PWM): now also TP10.1
- net at U1.P11 (RESERVED8): now also R31.2
- net at U2.P11 (RESERVED8): now also R32.2
