File: Design/Projector/DLP_Board/dlp_01/dlp_01_sch_brd/dlp_controller_config.sch (KiCad schematic (older format))
At the start: 51 parts, among them U1 DLPC3437, U2 DLPC3437, U3 ASDMB-24.000MHZ-LC-T, U4 W25Q64JVSSIQ, U5 W25Q64JVSSIQ

Commit message: Dump of uncommitted changes
Parts:
- added TP11: TestPoint, TestPoint:TestPoint_Pad_D1.5mm, symbol Connector:TestPoint
- C100, C47, C99: footprint Capacitors_SMD:C_0603 -> Capacitor_SMD:C_0603_1608Metric; part-num (none) -> 06033C104KAT4A
- R14, R15, R22, R26, R30, R33, R34, R40: footprint Resistors_SMD:R_0603 -> Resistor_SMD:R_0603_1608Metric; part-num (none) -> CRCW0603100KFKEA
- R16, R20, R23, R25, R27, R38, R41, R43, R44: footprint Resistors_SMD:R_0603 -> Resistor_SMD:R_0603_1608Metric; part-num (none) -> CRCW060330R1FKEA
- R17, R18, R28, R29, R35, R36, R46, R47: footprint Resistors_SMD:R_0603 -> Resistor_SMD:R_0603_1608Metric; part-num (none) -> CRCW06030000Z0EAC
- R19, R37, R45: footprint Resistors_SMD:R_0603 -> Resistor_SMD:R_0603_1608Metric; part-num (none) -> CRCW060310K0FKEA
- R21, R24, R39, R42: footprint Resistors_SMD:R_0603 -> Resistor_SMD:R_0603_1608Metric; part-num (none) -> CRCW06032K00FKEA
- R31, R32: value 8k -> 8.2k; footprint Resistors_SMD:R_0603 -> Resistor_SMD:R_0603_1608Metric; part-num (none) -> CRCW06038K20FKEA
- TP10, TP2, TP3, TP4, TP5, TP6, TP7, TP8, TP9: footprint Measurement_Points:Measurement_Point_Round-SMD-Pad_Small -> TestPoint:TestPoint_Pad_D1.5mm; DNP (none) -> TRUE
- U1, U2: part-num (none) -> DLPC3437CZEZ
- U3: footprint Oscillators:Oscillator_SMD_SeikoEpson_SG210-4pin_2.5x2.0mm_HandSoldering -> Oscillator:Oscillator_SMD_SeikoEpson_SG210-4Pin_2.5x2.0mm_HandSoldering; symbol Oscillator:ASDMB-xxxMHz -> dlp_01-rescue:ASDMB-xxxMHz-Oscillator; part-num (none) -> ASDMB-24.000MHZ-LC-T
- U4, U5: footprint Housings_SOIC:SO-8_5.3x6.2mm_Pitch1.27mm -> Package_SO:SO-8_5.3x6.2mm_P1.27mm; symbol Memory_Flash:W25Q32JVSS -> dlp_01-rescue:W25Q32JVSS-Memory_Flash; part-num (none) -> W25Q64JVSSIQ
Connections:
- net +1V8: no longer U3.1 (Standby)
- net at U1.P11 (RESERVED8): now also R31.2
- net at U2.P11 (RESERVED8): now also R32.2
- new net: TP11.1, U3.1 (Standby)
Other:
- moved on the sheet: C47, R16, U3
