File: Design/Projector/DLP_Board/dlp_01/dlp_01_sch_brd/dlp_controller_dmdinterface.sch (KiCad schematic (older format))
At the start: 4 parts, among them U1 DLPC3437, U2 DLPC3437

Commit message: Dump of uncommitted changes
Parts:
- R52, R53: footprint Resistors_SMD:R_0603 -> Resistor_SMD:R_0603_1608Metric; part-num (none) -> CRCW060343R0FKEA
- U1, U2: part-num (none) -> DLPC3437CZEZ
Changed lines of the file:
@@
 EESchema Schematic File Version 4
-EELAYER 30 0
+LIBS:dlp_01-cache
+EELAYER 26 0
 EELAYER END
 $Descr A3 16535 11693
@@
 F 2 "ZEZ0201A:BGA-225_15x15_13.1x13.1mm" H 6300 4000 50  0001 C CNN
 F 3 "http://www.ti.com/lit/ds/symlink/dlpc3437.pdf" H 5300 3650 50  0001 C CNN
+F 4 "DLPC3437CZEZ" H 0   0   50  0001 C CNN "part-num"
 	2    5300 3650
 	1    0    0    -1
@@
 F 2 "ZEZ0201A:BGA-225_15x15_13.1x13.1mm" H 6300 2950 50  0001 C CNN
 F 3 "http://www.ti.com/lit/ds/symlink/dlpc3437.pdf" H 5300 2600 50  0001 C CNN
+F 4 "DLPC3437CZEZ" H 0   0   50  0001 C CNN "part-num"
 	3    5300 2600
 	1    0    0    -1
@@
 F 0 "R52" V 4441 2400 50  0000 C CNN
 F 1 "43R" V 4532 2400 50  0000 C CNN
-F 2 "Resistors_SMD:R_0603" V 4604 2400 25  0000 C CNN
+F 2 "Resistor_SMD:R_0603_1608Metric" V 4604 2400 25  0000 C CNN
 F 3 "~" H 4700 2400 50  0001 C CNN
+F 4 "CRCW060343R0FKEA" H 0   0   50  0001 C CNN "part-num"
 	1    4700 2400
 	0    1    1    0
@@
 F 0 "R53" V 4441 2800 50  0000 C CNN
 F 1 "43R" V 4532 2800 50  0000 C CNN
-F 2 "Resistors_SMD:R_0603" V 4604 2800 25  0000 C CNN
+F 2 "Resistor_SMD:R_0603_1608Metric" V 4604 2800 25  0000 C CNN
 F 3 "~" H 4700 2800 50  0001 C CNN
+F 4 "CRCW060343R0FKEA" H 0   0   50  0001 C CNN "part-num"
 	1    4700 2800
 	0    1    1    0
@@
 F 2 "ZEZ0201A:BGA-225_15x15_13.1x13.1mm" H 11600 4000 50  0001 C CNN
 F 3 "http://www.ti.com/lit/ds/symlink/dlpc3437.pdf" H 10600 3650 50  0001 C CNN
+F 4 "DLPC3437CZEZ" H 0   0   50  0001 C CNN "part-num"
 	2    10600 3650
 	1    0    0    -1
@@
 F 2 "ZEZ0201A:BGA-225_15x15_13.1x13.1mm" H 11600 3000 50  0001 C CNN
 F 3 "http://www.ti.com/lit/ds/symlink/dlpc3437.pdf" H 10600 2650 50  0001 C CNN
+F 4 "DLPC3437CZEZ" H 0   0   50  0001 C CNN "part-num"
 	3    10600 2650
 	1    0    0    -1
