File: Design/Projector/DLP_Board/dlp_01/dlp_01_sch_brd/dlp_pmic.sch (KiCad schematic (older format))
At the start: 59 parts

Commit message: Initial placement of power converters, BGA fanout and Z-turn board outline imported
Parts:
- added R54, R55, R59, R62: NF, Resistors_SMD:R_0603, symbol Device:R
- C64: renamed from C?; value 10u -> 1u
- D1: renamed from D?; footprint Diode_SMD:D_SOD-123 -> Diodes_SMD:D_SOD-123
- gave numbers to parts that had none: 56
Connections:
- net +1V1: now also R54.1; no longer C48.2, C50.2, L1.1, U6.94 (PWR1_FB)
- net +1V8: now also R55.1; no longer C49.2, C51.2, L2.1, U6.72 (PWR2_FB)
- net +2V5: now also R59.2; no longer C61.2, U6.87 (PWR3_OUT)
- net +3V3: now also R62.2; no longer C72.2, U6.89 (PWR4_OUT)
- net GND: now also U6.93 (PWR1_PGND)
- net VBIAS: no longer C67.2
- net VOFS: now also C67.2
- net LEDx_CATHODE: now reaches R64.2, U6.11 (RLIM_1), U6.13 (RLIM_K_2), U6.15 (RLIM_K_1), U6.16 (RLIM_1), U6.22 (RLIM_2), U6.23 (RLIM_2)
- net +19V renamed +12V
- net ILLUM_5P5V: no longer names the net of C84.2, U6.7 (ILLUM_5P5V)
- net PWR_5P5V: no longer names the net of C76.2, U6.84 (PWR_5P5V)
- new net: C72.2, R62.1, U6.89 (PWR4_OUT)
- new net: C61.2, R59.1, U6.87 (PWR3_OUT)
- new net: C49.2, C51.2, L2.1, R55.2, U6.72 (PWR2_FB)
- new net: C48.2, C50.2, L1.1, R54.2, U6.94 (PWR1_FB)
- no-connect marks 23 -> 25
