File: Design/Projector/DLP_Board/dlp_01/dlp_01_sch_brd/dlp_pmic.sch (KiCad schematic (older format))
At the start: 62 parts, among them U6 DLPA3000

Commit message: Dump of uncommitted changes
Parts:
- added R102: 0R, Resistor_SMD:R_0805_2012Metric, symbol Device:R
- added R81, R82: NF, Resistor_SMD:R_0603_1608Metric, symbol Device:R
- C48, C49, C50, C51, C52, C53, C55, C56, C77, C80, C83, C85, C86, C88: footprint Capacitors_SMD:C_1206 -> Capacitor_SMD:C_1206_3216Metric; part-num (none) -> 12063D226MAT2A
- C54, C70, C74, C75: footprint Capacitors_SMD:C_0603 -> Capacitor_SMD:C_0603_1608Metric; part-num (none) -> 06033C104KAT4A
- C57, C60, C61, C64, C66, C72, C81, C87: footprint Capacitors_SMD:C_1206 -> Capacitor_SMD:C_1206_3216Metric; part-num (none) -> 12065C105KAZ4A
- C58, C67: footprint Capacitors_SMD:C_0603 -> Capacitor_SMD:C_0603_1608Metric; Voltage (none) -> 50V; part-num (none) -> GRT188R61H105KE13D
- C59, C71, C76, C84: footprint Capacitors_SMD:C_1206 -> Capacitor_SMD:C_1206_3216Metric; part-num (none) -> 12065D106KAT2A
- C62: footprint Capacitors_SMD:C_0603 -> Capacitor_SMD:C_0603_1608Metric; Voltage (none) -> 50V; part-num (none) -> C1608X7R1H474K080AC
- C63: footprint Capacitors_SMD:C_0603 -> Capacitor_SMD:C_0603_1608Metric; part-num (none) -> GRT188R61H105KE13D
- C65: footprint Capacitors_SMD:C_1206 -> Capacitor_SMD:C_1206_3216Metric; part-num (none) -> 12065C225K4T2A
- C68, C69: value 100n -> 470p; footprint Capacitors_SMD:C_0603 -> Capacitor_SMD:C_0603_1608Metric; part-num (none) -> 06033C471KAT4A
- C73: footprint Capacitors_SMD:C_1206 -> Capacitor_SMD:C_1206_3216Metric; part-num (none) -> 12065C475KAT4A
- C78: value 1.2n -> 10p; footprint Capacitors_SMD:C_0603 -> Capacitor_SMD:C_0603_1608Metric; part-num (none) -> 06033C100KAT2A
- C79, C82: footprint Capacitors_SMD:C_0603 -> Capacitor_SMD:C_0603_1608Metric; part-num (none) -> 06033C122KAT2A
- D1: footprint Diodes_SMD:D_SOD-123 -> Diode_SMD:D_SOD-123; part-num (none) -> MBR0540
- D2, D3, D4: footprint Diodes_SMD:D_SOD-523 -> Diode_SMD:D_SOD-523; part-num (none) -> ESDA18-1K
- L1, L2: footprint Inductors_SMD:L_Taiyo-Yuden_MD-2020 -> Inductor_SMD:L_Taiyo-Yuden_MD-2020; part-num (none) -> IHLP2020BZER3R3M11
- L3: footprint Coilcraft:L_Coilcraft_LPS4018 -> Inductor_SMD:L_Coilcraft_LPS4018; part-num (none) -> LPS4018-103MRB
- L4: part-num (none) -> XAL7030-272MEB
- R54, R55, R59, R62: footprint Resistors_SMD:R_0603 -> Resistor_SMD:R_0603_1608Metric; DNP (none) -> TRUE; part-num (none) -> NF
- R56: footprint Resistors_SMD:R_0603 -> Resistor_SMD:R_0603_1608Metric; part-num (none) -> CRCW0603300RFKEA
- R57: footprint Resistors_SMD:R_0603 -> Resistor_SMD:R_0603_1608Metric; part-num (none) -> CRCW06035K10FKEA
- R58: footprint Resistors_SMD:R_0603 -> Resistor_SMD:R_0603_1608Metric; part-num (none) -> CRCW060310K0FKEA
- R60, R61: footprint Resistors_SMD:R_0603 -> Resistor_SMD:R_0603_1608Metric; part-num (none) -> CRCW060310R0FKEA
- R63: footprint Resistors_SMD:R_0603 -> Resistor_SMD:R_0603_1608Metric; part-num (none) -> CRCW060330R1FKEA
- R64: footprint Resistors_SMD:R_2010 -> Resistor_SMD:R_2010_5025Metric; part-num (none) -> CRCW20100000Z0EF
- R65: footprint Resistors_SMD:R_0603 -> Resistor_SMD:R_0603_1608Metric; part-num (none) -> CRCW06033R90FKEA
- U6: footprint HTQFP-100:HTQFP-100_14x14mm_Pitch0.5mm_EP -> Package_QFP:TQFP-100-1EP_14x14mm_P0.5mm_EP5x5mm; part-num (none) -> DLPA3000DPFD
Connections:
- net GND: now also U6.37 (ILLUM_B_PGND), R81.2, R82.2
- net SPI1_CLK: now also R82.1
- net SPI1_DOUT: now also R81.1
- net at C79.2, C82.2, L4.1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: now also R102.2
- net at U6.36 (ILLUM_B_SW): now also R102.1
- no-connect marks 25 -> 23
Other:
- moved on the sheet: C82, C85, C88, L4, R65
