File: Design/Projector/DLP_Board/dlp_01/dlp_01_sch_brd/dlp_controller_power.sch (KiCad schematic (older format))
At the start: 52 parts

Commit message: Initial placement of power converters, BGA fanout and Z-turn board outline imported
Parts:
- gave numbers to parts that had none: 52

Commit message: Initial component placement on PCB
Parts:
- C1, C10, C11, C12, C13, C14, C15, C16, C17, C18, C19, C2, C20, C21, C22, C23, C24, C25, C26, C27, C28, C29, C3, C30, C31, C32, C33, C34, C35, C36, C37, C38, C39, C4, C40, C41, C42, C43, C44, C45, C46, C5, C6, C7, C8, C9: footprint Capacitors_SMD:C_0603 -> Capacitors_SMD:C_0402
- FB1, FB2, FB3, FB4: value BLM18KG121TN1D -> BLM15PD800SN1D; footprint Inductors_SMD:L_0603 -> Inductors_SMD:L_0402
Connections:
- net +1V1: no longer C12.1, C13.1, C15.1, C16.1, C18.1, C19.1, C21.1, C22.1, C24.1, C25.1, C26.1, C27.1, C29.1, C3.1, C30.1, C34.1, C35.1, C38.1, C39.1, C4.1, C41.1, C42.1, C8.1, C9.1
- net +1V8: now also C12.1, C13.1, C15.1, C16.1, C18.1, C19.1, C21.1, C22.1, C24.1, C25.1, C26.1, C27.1, C29.1, C3.1, C30.1, C34.1, C35.1, C38.1, C39.1, C4.1, C41.1, C42.1, C8.1, C9.1
