File: Design/Projector/DLP_Board/dlp_01/dlp_01_sch_brd/dlp_controller_power.sch (KiCad schematic (older format))
At the start: 52 parts, among them U1 DLPC3437, U2 DLPC3437

Commit message: Dump of uncommitted changes
Parts:
- C1, C10, C11, C12, C13, C14, C15, C16, C17, C18, C19, C2, C20, C21, C22, C23, C24, C25, C26, C27, C28, C29, C3, C30, C31, C32, C34, C35, C36, C37, C38, C39, C4, C40, C41, C42, C43, C44, C45, C46, C5, C7, C8, C9: footprint Capacitors_SMD:C_0402 -> Capacitor_SMD:C_0402_1005Metric; part-num (none) -> 0402ZD104KAT2A
- C33, C6: footprint Capacitors_SMD:C_0402 -> Capacitor_SMD:C_0402_1005Metric; part-num (none) -> 0402ZD103KAT2A
- FB1, FB2, FB3, FB4: footprint Inductors_SMD:L_0402 -> Inductor_SMD:L_0402_1005Metric; part-num (none) -> BLM15PD800SN1D
- U1, U2: part-num (none) -> DLPC3437CZEZ
