File: Design/Projector/DLP_Board/dlp_01/dlp_01_sch_brd/power.sch (KiCad schematic (older format))
At the start: 14 parts, among them J10 Screw_Terminal_01x03, J3 Barrel_Jack_MountingPin, Q1 2N7000, U8 RPM5.0-3.0

Commit message: Schematic and PCB complete ready for review
Parts:
- removed J10: Screw_Terminal_01x03, Connectors_Terminal_Blocks:TerminalBlock_bornier-3_P5.08mm, symbol Connector:Screw_Terminal_01x03
Connections:
- net GND: now also J3.3 (MountPin)
- no-connect marks 3 -> 1
Changed lines of the file:
@@
 	1    0    0    -1
 $EndComp
-NoConn ~ 1800 3500
 Wire Wire Line
 	2550 3650 2550 3300
@@
 	1    0    0    -1
 $EndComp
-$Comp
-L Connector:Screw_Terminal_01x03 J?
-U 1 1 5DF838E9
-P 1750 2600
-AR Path="/5DF838E9" Ref="J?"  Part="1"
-AR Path="/5D37DB5E/5DF838E9" Ref="J10"  Part="1"
-F 0 "J10" H 1668 2969 50  0000 C CNN
-F 1 "Screw_Terminal_01x03" H 1668 2878 50  0000 C CNN
-F 2 "Connectors_Terminal_Blocks:TerminalBlock_bornier-3_P5.08mm" H 1668 2806 25  0000 C CNN
-F 3 "~" H 1750 2600 50  0001 C CNN
-	1    1750 2600
-	-1   0    0    -1
-$EndComp
-Wire Wire Line
-	2100 3100 2800 3100
 Connection ~ 3150 3100
 Wire Wire Line
-	1950 2500 2800 2500
-Wire Wire Line
-	2800 2500 2800 3100
-Connection ~ 2800 3100
-Wire Wire Line
-	2800 3100 3150 3100
-Wire Wire Line
 	2100 3300 2550 3300
 Wire Wire Line
-	2550 3300 2550 2700
-Wire Wire Line
-	2550 2700 1950 2700
-Connection ~ 2550 3300
-NoConn ~ 1950 2600
+	2100 3100 3150 3100
+$Comp
+L power:GND #PWR0142
+U 1 1 5D8D24F6
+P 1800 3650
+F 0 "#PWR0142" H 1800 3400 50  0001 C CNN
+F 1 "GND" H 1805 3477 50  0000 C CNN
+F 2 "" H 1800 3650 50  0001 C CNN
+F 3 "" H 1800 3650 50  0001 C CNN
+	1    1800 3650
+	1    0    0    -1
+$EndComp
+Wire Wire Line
+	1800 3500 1800 3650
 $EndSCHEMATC
