File: Design/Projector/DLP_Board/dlp_01/dlp_01_sch_brd/application_connectors.sch (KiCad schematic (older format))
At the start: 15 parts, among them J1 Conn_02x40_Odd_Even, J2 Conn_02x40_Odd_Even

Commit message: Dump of uncommitted changes
Parts:
- removed R81, R82: NF, Resistors_SMD:R_0603, symbol Device:R
- added J10: NF_SFM-140-02-S-D-LC, Connector_PinSocket_1.27mm:PinSocket_2x40_P1.27mm_Vertical_SMD, symbol Connector_Generic:Conn_02x40_Odd_Even
- added R103, R104, R105, R106, R107, R108, R109, R110, R111, R112, R113, R114, R115: NF, Resistor_SMD:R_0603_1608Metric, symbol Device:R
- J1, J2: value Conn_02x40_Odd_Even -> FTSH-140-01-F-DV-P; footprint Pin_Headers:Pin_Header_Straight_2x40_Pitch1.27mm_SMD -> Connector_PinHeader_1.27mm:PinHeader_2x40_P1.27mm_Vertical_SMD; part-num (none) -> FTSH-140-01-F-DV-P
- R68, R69, R70, R71, R72, R73, R74, R77, R78, R80, R89: footprint Resistors_SMD:R_0603 -> Resistor_SMD:R_0603_1608Metric; DNP (none) -> TRUE; part-num (none) -> NF
Connections:
- net labels removed: PL_SCL, PL_SDA, PS_SCL, PS_SDA
- wire segments 252 -> 346
- no-connect marks 3 -> 4
Other:
- note added: "Extension of MYiR Z-Turn Board Connector"
- moved on the sheet: J1, J2, R68, R69, R70, R71, R72, R73, R74, R77, R78, R80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
