File: Design/Projector/DLP_Board/dlp_01/dlp_01_sch_brd/dlp_01.sch (KiCad schematic (older format))
At the start: 12 parts, among them J4 Screw_Terminal_01x03, J5 Screw_Terminal_01x03, J6 Conn_01x03_Male, J7 Conn_01x03_Male, J8 Conn_01x03_Male, J9 Conn_01x03_Male

Commit message: Dump of uncommitted changes
Parts:
- H1, H2, H3, H4, H5, H6: footprint Mounting_Holes:MountingHole_3mm_Pad_Via -> MountingHole:MountingHole_3.2mm_M3_Pad_Via; DNP (none) -> TRUE
- J4, J5: footprint Connectors_Terminal_Blocks:TerminalBlock_bornier-3_P5.08mm -> TerminalBlock:TerminalBlock_bornier-3_P5.08mm; part-num (none) -> TB006-508-03BE
- J6, J7, J8, J9: footprint Pin_Headers:Pin_Header_Straight_1x03_Pitch2.54mm_SMD_Pin1Left -> Connector_PinHeader_2.54mm:PinHeader_1x03_P2.54mm_Vertical_SMD_Pin1Left; part-num (none) -> 87898-0306
Connections:
- no-connect marks 5 -> 1
Changed lines of the file:
@@
 EESchema Schematic File Version 4
-EELAYER 30 0
+LIBS:dlp_01-cache
+EELAYER 26 0
 EELAYER END
 $Descr A3 16535 11693
@@
 F5 "DATEN_B" O R 6900 4250 50
 F6 "PDAT_B_[23..0]" O R 6900 4100 50
-F7 "3DR_B" O R 6900 4300 50
-F8 "PCLK_A" O R 6900 3600 50
-F9 "VSYNC_A" O R 6900 3700 50
-F10 "HSYNC_A" O R 6900 3750 50
-F11 "DATEN_A" O R 6900 3800 50
-F12 "PDAT_A_[23..0]" O R 6900 3650 50
-F13 "3DR_A" O R 6900 3850 50
-F14 "PDM_CVS_TE_B" I R 6900 4350 50
-F15 "PDM_CVS_TE_A" I R 6900 3900 50
-F16 "HOST_SCL" O R 6900 2500 50
-F17 "HOST_SDA" B R 6900 2550 50
-F18 "CONTR0_SCL" O R 6900 2700 50
-F19 "CONTR0_SDA" B R 6900 2750 50
-F20 "CONTR1_SDA" B R 6900 2950 50
-F21 "CONTR1_SCL" O R 6900 2900 50
-F22 "PS_SCL" O R 6900 2100 50
-F23 "PL_SCL" O R 6900 2150 50
-F24 "PL_SDA" B R 6900 2300 50
-F25 "PS_SDA" B R 6900 2350 50
-F26 "FPGA_RDY" O R 6900 4700 50
-F27 "ACT_SYNC" I R 6900 4650 50
-F28 "SUB_FRAME" O R 6900 4600 50
-F29 "mHOST_IRQ" I R 6900 5000 50
-F30 "sHOST_IRQ" I R 6900 5050 50
-F31 "PROJ_ON" O R 6900 5200 50
+F7 "PCLK_A" O R 6900 3600 50
+F8 "VSYNC_A" O R 6900 3700 50
+F9 "HSYNC_A" O R 6900 3750 50
+F10 "DATEN_A" O R 6900 3800 50
+F11 "PDAT_A_[23..0]" O R 6900 3650 50
+F12 "PDM_CVS_TE_B" I R 6900 4350 50
+F13 "PDM_CVS_TE_A" I R 6900 3900 50
+F14 "HOST_SCL" O R 6900 2500 50
+F15 "HOST_SDA" B R 6900 2550 50
+F16 "CONTR0_SCL" O R 6900 2700 50
+F17 "CONTR0_SDA" B R 6900 2750 50
+F18 "CONTR1_SDA" B R 6900 2950 50
+F19 "CONTR1_SCL" O R 6900 2900 50
+F20 "FPGA_RDY" O R 6900 4700 50
+F21 "ACT_SYNC" I R 6900 4650 50
+F22 "SUB_FRAME" O R 6900 4600 50
+F23 "mHOST_IRQ" I R 6900 5000 50
+F24 "sHOST_IRQ" I R 6900 5050 50
+F25 "PROJ_ON" O R 6900 5200 50
 $EndSheet
 Wire Wire Line
@@
 Wire Wire Line
 	6900 4350 7550 4350
-NoConn ~ 6900 2100
-NoConn ~ 6900 2150
-NoConn ~ 6900 2300
-NoConn ~ 6900 2350
 Wire Wire Line
 	6900 2500 7550 2500
@@
 F 0 "J4" H 4368 7569 50  0000 C CNN
 F 1 "Screw_Terminal_01x03" H 4368 7478 50  0000 C CNN
-F 2 "Connectors_Terminal_Blocks:TerminalBlock_bornier-3_P5.08mm" H 4368 7406 25  0000 C CNN
+F 2 "TerminalBlock:TerminalBlock_bornier-3_P5.08mm" H 4368 7406 25  0000 C CNN
 F 3 "~" H 4450 7200 50  0001 C CNN
+F 4 "TB006-508-03BE" H 0   0   50  0001 C CNN "part-num"
 	1    4450 7200
 	-1   0    0    -1
@@
 F 0 "J5" H 4368 8669 50  0000 C CNN
 F 1 "Screw_Terminal_01x03" H 4368 8578 50  0000 C CNN
-F 2 "Connectors_Terminal_Blocks:TerminalBlock_bornier-3_P5.08mm" H 4368 8506 25  0000 C CNN
+F 2 "TerminalBlock:TerminalBlock_bornier-3_P5.08mm" H 4368 8506 25  0000 C CNN
 F 3 "~" H 4450 8300 50  0001 C CNN
+F 4 "TB006-508-03BE" H 0   0   50  0001 C CNN "part-num"
 	1    4450 8300
 	-1   0    0    -1
@@
 F 0 "J6" H 14172 2850 50  0000 R CNN
 F 1 "Conn_01x03_Male" H 14172 2759 50  0000 R CNN
-F 2 "Pin_Headers:Pin_Header_Straight_1x03_Pitch2.54mm_SMD_Pin1Left" H 14172 2687 25  0000 R CNN
+F 2 "Connector_PinHeader_2.54mm:PinHeader_1x03_P2.54mm_Vertical_SMD_Pin1Left" H 14172 2687 25  0000 R CNN
 F 3 "~" H 14200 2800 50  0001 C CNN
+F 4 "87898-0306" H 14200 2800 50  0001 C CNN "part-num"
 	1    14200 2800
 	-1   0    0    -1
@@
 F 0 "J7" H 14172 3700 50  0000 R CNN
 F 1 "Conn_01x03_Male" H 14172 3609 50  0000 R CNN
-F 2 "Pin_Headers:Pin_Header_Straight_1x03_Pitch2.54mm_SMD_Pin1Left" H 14172 3537 25  0000 R CNN
+F 2 "Connector_PinHeader_2.54mm:PinHeader_1x03_P2.54mm_Vertical_SMD_Pin1Left" H 14172 3537 25  0000 R CNN
 F 3 "~" H 14200 3650 50  0001 C CNN
+F 4 "87898-0306" H 0   0   50  0001 C CNN "part-num"
 	1    14200 3650
 	-1   0    0    -1
@@
 F 0 "J8" H 14172 4600 50  0000 R CNN
 F 1 "Conn_01x03_Male" H 14172 4509 50  0000 R CNN
-F 2 "Pin_Headers:Pin_Header_Straight_1x03_Pitch2.54mm_SMD_Pin1Left" H 14172 4437 25  0000 R CNN
+F 2 "Connector_PinHeader_2.54mm:PinHeader_1x03_P2.54mm_Vertical_SMD_Pin1Left" H 14172 4437 25  0000 R CNN
 F 3 "~" H 14200 4550 50  0001 C CNN
+F 4 "87898-0306" H 0   0   50  0001 C CNN "part-num"
 	1    14200 4550
 	-1   0    0    -1
@@
 F 0 "J9" H 14172 5450 50  0000 R CNN
 F 1 "Conn_01x03_Male" H 14172 5359 50  0000 R CNN
-F 2 "Pin_Headers:Pin_Header_Straight_1x03_Pitch2.54mm_SMD_Pin1Left" H 14172 5287 25  0000 R CNN
+F 2 "Connector_PinHeader_2.54mm:PinHeader_1x03_P2.54mm_Vertical_SMD_Pin1Left" H 14172 5287 25  0000 R CNN
 F 3 "~" H 14200 5400 50  0001 C CNN
+F 4 "87898-0306" H 0   0   50  0001 C CNN "part-num"
 	1    14200 5400
 	-1   0    0    -1
@@
 F 0 "H1" H 1100 10099 50  0000 L CNN
 F 1 "3mm" H 1100 10008 50  0000 L CNN
-F 2 "Mounting_Holes:MountingHole_3mm_Pad_Via" H 1000 10050 50  0001 C CNN
+F 2 "MountingHole:MountingHole_3.2mm_M3_Pad_Via" H 1000 10050 50  0001 C CNN
 F 3 "~" H 1000 10050 50  0001 C CNN
+F 4 "TRUE" H 0   0   50  0001 C CNN "DNP"
 	1    1000 10050
 	1    0    0    -1
@@
 F 0 "H2" H 1500 10099 50  0000 L CNN
 F 1 "3mm" H 1500 10008 50  0000 L CNN
-F 2 "Mounting_Holes:MountingHole_3mm_Pad_Via" H 1400 10050 50  0001 C CNN
+F 2 "MountingHole:MountingHole_3.2mm_M3_Pad_Via" H 1400 10050 50  0001 C CNN
 F 3 "~" H 1400 10050 50  0001 C CNN
+F 4 "TRUE" H 0   0   50  0001 C CNN "DNP"
 	1    1400 10050
 	1    0    0    -1
@@
 F 0 "H3" H 1900 10099 50  0000 L CNN
 F 1 "3mm" H 1900 10008 50  0000 L CNN
-F 2 "Mounting_Holes:MountingHole_3mm_Pad_Via" H 1800 10050 50  0001 C CNN
+F 2 "MountingHole:MountingHole_3.2mm_M3_Pad_Via" H 1800 10050 50  0001 C CNN
 F 3 "~" H 1800 10050 50  0001 C CNN
+F 4 "TRUE" H 0   0   50  0001 C CNN "DNP"
 	1    1800 10050
 	1    0    0    -1
@@
 F 0 "H4" H 2300 10099 50  0000 L CNN
 F 1 "3mm" H 2300 10008 50  0000 L CNN
-F 2 "Mounting_Holes:MountingHole_3mm_Pad_Via" H 2200 10050 50  0001 C CNN
+F 2 "MountingHole:MountingHole_3.2mm_M3_Pad_Via" H 2200 10050 50  0001 C CNN
 F 3 "~" H 2200 10050 50  0001 C CNN
+F 4 "TRUE" H 0   0   50  0001 C CNN "DNP"
 	1    2200 10050
 	1    0    0    -1
@@
 F 0 "H5" H 2700 10099 50  0000 L CNN
 F 1 "3mm" H 2700 10008 50  0000 L CNN
-F 2 "Mounting_Holes:MountingHole_3mm_Pad_Via" H 2600 10050 50  0001 C CNN
+F 2 "MountingHole:MountingHole_3.2mm_M3_Pad_Via" H 2600 10050 50  0001 C CNN
 F 3 "~" H 2600 10050 50  0001 C CNN
+F 4 "TRUE" H 0   0   50  0001 C CNN "DNP"
 	1    2600 10050
 	1    0    0    -1
@@
 F 0 "H6" H 3100 10099 50  0000 L CNN
 F 1 "3mm" H 3100 10008 50  0000 L CNN
-F 2 "Mounting_Holes:MountingHole_3mm_Pad_Via" H 3000 10050 50  0001 C CNN
+F 2 "MountingHole:MountingHole_3.2mm_M3_Pad_Via" H 3000 10050 50  0001 C CNN
 F 3 "~" H 3000 10050 50  0001 C CNN
+F 4 "TRUE" H 0   0   50  0001 C CNN "DNP"
 	1    3000 10050
 	1    0    0    -1
