File: Design/Projector/DLP_Board/dlp_01/dlp_01_sch_brd/dlp_controller.sch (KiCad schematic (older format))
At the start: 0 parts

Commit message: Dump of uncommitted changes
Parts:
- added R100, R75, R76, R83, R84, R86, R87, R90: NF, Resistor_SMD:R_0603_1608Metric, symbol Device:R
- added R101, R79, R85, R88: 0R, Resistor_SMD:R_0603_1608Metric, symbol Device:R
Connections:
- net SPI1_CLK: now also R75.1, R76.1, R79.1
- net SPI1_CSZ0: now also R100.1, R101.1, R90.1
- net SPI1_DIN: now also R83.1, R84.1, R85.1
- net SPI1_DOUT: now also R86.1, R87.1, R88.1
- net dlp_controller_config/mSPI_CLK: now also R75.2
- net dlp_controller_config/mSPI_CSZO: now also R90.2
- net dlp_controller_config/mSPI_MISO: now also R86.2
- net dlp_controller_config/mSPI_MOSI: now also R83.2
- net dlp_controller_config/sSPI_CLK: now also R76.2
- net dlp_controller_config/sSPI_CSZO: now also R100.2
- net dlp_controller_config/sSPI_MISO: now also R87.2
- net dlp_controller_config/sSPI_MOSI: now also R84.2
- new net dlp_controller_gpio/SPI1_CLK: R79.2
- new net dlp_controller_gpio/SPI1_CSZ0: R101.2
- new net dlp_controller_gpio/SPI1_DIN: R85.2
- new net dlp_controller_gpio/SPI1_DOUT: R88.2
- no-connect marks 8 -> 0
