File: Design/Projector/DLP_Board/dlp_01/dlp_01_sch_brd/dlp_controller_datainterface.sch (KiCad schematic (older format))
At the start: 6 parts, among them U1 DLPC3437, U2 DLPC3437

Commit message: Dump of uncommitted changes
Parts:
- R48, R49, R50, R51: footprint Resistors_SMD:R_0603 -> Resistor_SMD:R_0603_1608Metric; part-num (none) -> CRCW06037K87FKEA
- U1, U2: part-num (none) -> DLPC3437CZEZ
Changed lines of the file:
@@
 EESchema Schematic File Version 4
-EELAYER 30 0
+LIBS:dlp_01-cache
+EELAYER 26 0
 EELAYER END
 $Descr A3 16535 11693
@@
 F 0 "R48" H 5970 7422 50  0000 L CNN
 F 1 "7.87k" H 5970 7331 50  0000 L CNN
-F 2 "Resistors_SMD:R_0603" H 5970 7259 25  0000 L CNN
+F 2 "Resistor_SMD:R_0603_1608Metric" H 5970 7259 25  0000 L CNN
 F 3 "~" H 5900 7350 50  0001 C CNN
+F 4 "CRCW06037K87FKEA" H 0   0   50  0001 C CNN "part-num"
 	1    5900 7350
 	1    0    0    -1
@@
 F 0 "R49" V 5841 3500 50  0000 C CNN
 F 1 "7.87k" V 5932 3500 50  0000 C CNN
-F 2 "Resistors_SMD:R_0603" V 6004 3500 25  0000 C CNN
+F 2 "Resistor_SMD:R_0603_1608Metric" V 6004 3500 25  0000 C CNN
 F 3 "~" H 6100 3500 50  0001 C CNN
+F 4 "CRCW06037K87FKEA" H 0   0   50  0001 C CNN "part-num"
 	1    6100 3500
 	0    1    1    0
@@
 F 2 "ZEZ0201A:BGA-225_15x15_13.1x13.1mm" H 7250 4450 50  0001 C CNN
 F 3 "http://www.ti.com/lit/ds/symlink/dlpc3437.pdf" H 6250 4100 50  0001 C CNN
+F 4 "DLPC3437CZEZ" H 0   0   50  0001 C CNN "part-num"
 	4    6250 4100
 	1    0    0    -1
@@
 F 0 "R50" H 9970 7422 50  0000 L CNN
 F 1 "7.87k" H 9970 7331 50  0000 L CNN
-F 2 "Resistors_SMD:R_0603" H 9970 7259 25  0000 L CNN
+F 2 "Resistor_SMD:R_0603_1608Metric" H 9970 7259 25  0000 L CNN
 F 3 "~" H 9900 7350 50  0001 C CNN
+F 4 "CRCW06037K87FKEA" H 0   0   50  0001 C CNN "part-num"
 	1    9900 7350
 	1    0    0    -1
@@
 F 0 "R51" V 9841 3500 50  0000 C CNN
 F 1 "7.87k" V 9932 3500 50  0000 C CNN
-F 2 "Resistors_SMD:R_0603" V 10004 3500 25  0000 C CNN
+F 2 "Resistor_SMD:R_0603_1608Metric" V 10004 3500 25  0000 C CNN
 F 3 "~" H 10100 3500 50  0001 C CNN
+F 4 "CRCW06037K87FKEA" H 0   0   50  0001 C CNN "part-num"
 	1    10100 3500
 	0    1    1    0
@@
 F 2 "ZEZ0201A:BGA-225_15x15_13.1x13.1mm" H 11250 4450 50  0001 C CNN
 F 3 "http://www.ti.com/lit/ds/symlink/dlpc3437.pdf" H 10250 4100 50  0001 C CNN
+F 4 "DLPC3437CZEZ" H 0   0   50  0001 C CNN "part-num"
 	4    10250 4100
 	1    0    0    -1
