File: Design/Projector/DLP_Board/dlp_01/dlp_01_sch_brd/dlp_controller_gpio.sch (KiCad schematic (older format))
At the start: 26 parts, among them U1 DLPC3437, U2 DLPC3437, U9 NF_SN74AUP1T17

Commit message: Dump of uncommitted changes
Parts:
- C95, C96, C97, C98, TH1: footprint Capacitors_SMD:C_0603 -> Capacitor_SMD:C_0603_1608Metric; DNP (none) -> TRUE; part-num (none) -> NF
- R1, R2, R3: value 7.87k -> 30.1; footprint Resistors_SMD:R_0603 -> Resistor_SMD:R_0603_1608Metric; part-num (none) -> CRCW060330R1FKEA
- R10, R13, R4: footprint Resistors_SMD:R_0603 -> Resistor_SMD:R_0603_1608Metric; part-num (none) -> CRCW06037K87FKEA
- R11, R12, R5, R6: footprint Resistors_SMD:R_0603 -> Resistor_SMD:R_0603_1608Metric; part-num (none) -> CRCW060330R1FKEA
- R66, R67, R98, R99: footprint Resistors_SMD:R_0603 -> Resistor_SMD:R_0603_1608Metric; DNP (none) -> TRUE; part-num (none) -> NF
- R7, R8, R9: footprint Resistors_SMD:R_0603 -> Resistor_SMD:R_0603_1608Metric; part-num (none) -> CRCW0603100KFKEA
- TP1: footprint Measurement_Points:Measurement_Point_Round-SMD-Pad_Small -> TestPoint:TestPoint_Pad_D1.5mm; DNP (none) -> TRUE
- U1, U2: part-num (none) -> DLPC3437CZEZ
- U9: DNP (none) -> TRUE; part-num (none) -> SN74AUP1T17
Changed lines of the file:
@@
 EESchema Schematic File Version 4
-EELAYER 30 0
+LIBS:dlp_01-cache
+EELAYER 26 0
 EELAYER END
 $Descr A3 16535 11693
@@
 F 0 "R4" V 3791 7850 50  0000 C CNN
 F 1 "7.87k" V 3882 7850 50  0000 C CNN
-F 2 "Resistors_SMD:R_0603" V 3954 7850 25  0000 C CNN
+F 2 "Resistor_SMD:R_0603_1608Metric" V 3954 7850 25  0000 C CNN
 F 3 "~" H 4050 7850 50  0001 C CNN
+F 4 "CRCW06037K87FKEA" H 0   0   50  0001 C CNN "part-num"
 	1    4050 7850
 	0    1    1    0
@@
 F 0 "R5" V 3841 6050 50  0000 C CNN
 F 1 "30.1R" V 3932 6050 50  0000 C CNN
-F 2 "Resistors_SMD:R_0603" V 4004 6050 25  0000 C CNN
+F 2 "Resistor_SMD:R_0603_1608Metric" V 4004 6050 25  0000 C CNN
 F 3 "~" H 4100 6050 50  0001 C CNN
+F 4 "CRCW060330R1FKEA" H 0   0   50  0001 C CNN "part-num"
 	1    4100 6050
 	0    1    1    0
@@
 F 0 "R6" V 3841 6450 50  0000 C CNN
 F 1 "30.1R" V 3932 6450 50  0000 C CNN
-F 2 "Resistors_SMD:R_0603" V 4004 6450 25  0000 C CNN
+F 2 "Resistor_SMD:R_0603_1608Metric" V 4004 6450 25  0000 C CNN
 F 3 "~" H 4100 6450 50  0001 C CNN
+F 4 "CRCW060330R1FKEA" H 0   0   50  0001 C CNN "part-num"
 	1    4100 6450
 	0    1    1    0
@@
 F 2 "ZEZ0201A:BGA-225_15x15_13.1x13.1mm" H 6250 6700 50  0001 C CNN
 F 3 "http://www.ti.com/lit/ds/symlink/dlpc3437.pdf" H 5250 6350 50  0001 C CNN
+F 4 "DLPC3437CZEZ" H 0   0   50  0001 C CNN "part-num"
 	8    5250 6350
 	1    0    0    -1
@@
 F 0 "R11" V 5291 2000 50  0000 C CNN
 F 1 "30.1R" V 5382 2000 50  0000 C CNN
-F 2 "Resistors_SMD:R_0603" V 5454 2000 25  0000 C CNN
+F 2 "Resistor_SMD:R_0603_1608Metric" V 5454 2000 25  0000 C CNN
 F 3 "~" H 5550 2000 50  0001 C CNN
+F 4 "CRCW060330R1FKEA" H 0   0   50  0001 C CNN "part-num"
 	1    5550 2000
 	0    1    1    0
@@
 F 0 "R12" V 5291 2400 50  0000 C CNN
 F 1 "30.1R" V 5382 2400 50  0000 C CNN
-F 2 "Resistors_SMD:R_0603" V 5454 2400 25  0000 C CNN
+F 2 "Resistor_SMD:R_0603_1608Metric" V 5454 2400 25  0000 C CNN
 F 3 "~" H 5550 2400 50  0001 C CNN
+F 4 "CRCW060330R1FKEA" H 0   0   50  0001 C CNN "part-num"
 	1    5550 2400
 	0    1    1    0
@@
 F 2 "ZEZ0201A:BGA-225_15x15_13.1x13.1mm" H 7700 2650 50  0001 C CNN
 F 3 "http://www.ti.com/lit/ds/symlink/dlpc3437.pdf" H 6700 2300 50  0001 C CNN
+F 4 "DLPC3437CZEZ" H 0   0   50  0001 C CNN "part-num"
 	8    6700 2300
 	1    0    0    -1
@@
 F 0 "R13" V 5291 2800 50  0000 C CNN
 F 1 "7.87k" V 5382 2800 50  0000 C CNN
-F 2 "Resistors_SMD:R_0603" V 5454 2800 25  0000 C CNN
+F 2 "Resistor_SMD:R_0603_1608Metric" V 5454 2800 25  0000 C CNN
 F 3 "~" H 5550 2800 50  0001 C CNN
+F 4 "CRCW06037K87FKEA" H 0   0   50  0001 C CNN "part-num"
 	1    5550 2800
 	0    1    1    0
@@
 F 0 "TP1" V 6053 3772 50  0000 C CNN
 F 1 "TestPoint" V 6054 3772 50  0001 C CNN
-F 2 "Measurement_Points:Measurement_Point_Round-SMD-Pad_Small" H 6150 3700 50  0001 C CNN
+F 2 "TestPoint:TestPoint_Pad_D1.5mm" H 6150 3700 50  0001 C CNN
 F 3 "~" H 6150 3700 50  0001 C CNN
+F 4 "TRUE" H 0   0   50  0001 C CNN "DNP"
 	1    5950 3700
 	0    -1   -1   0
@@
 F 0 "R10" H 4880 3228 50  0000 R CNN
 F 1 "7.87k" H 4880 3319 50  0000 R CNN
-F 2 "Resistors_SMD:R_0603" H 4880 3391 25  0000 R CNN
+F 2 "Resistor_SMD:R_0603_1608Metric" H 4880 3391 25  0000 R CNN
 F 3 "~" H 4950 3300 50  0001 C CNN
+F 4 "CRCW06037K87FKEA" H 0   0   50  0001 C CNN "part-num"
 	1    4950 3300
 	-1   0    0    1
@@
 P 2300 3600
 F 0 "R1" V 2041 3600 50  0000 C CNN
-F 1 "7.87k" V 2132 3600 50  0000 C CNN
-F 2 "Resistors_SMD:R_0603" V 2204 3600 25  0000 C CNN
+F 1 "30.1" V 2132 3600 50  0000 C CNN
+F 2 "Resistor_SMD:R_0603_1608Metric" V 2204 3600 25  0000 C CNN
 F 3 "~" H 2300 3600 50  0001 C CNN
+F 4 "CRCW060330R1FKEA" H 0   0   50  0001 C CNN "part-num"
 	1    2300 3600
 	0    1    1    0
@@
 P 2300 4000
 F 0 "R2" V 2041 4000 50  0000 C CNN
-F 1 "7.87k" V 2132 4000 50  0000 C CNN
-F 2 "Resistors_SMD:R_0603" V 2204 4000 25  0000 C CNN
+F 1 "30.1" V 2132 4000 50  0000 C CNN
+F 2 "Resistor_SMD:R_0603_1608Metric" V 2204 4000 25  0000 C CNN
 F 3 "~" H 2300 4000 50  0001 C CNN
+F 4 "CRCW060330R1FKEA" H 0   0   50  0001 C CNN "part-num"
 	1    2300 4000
 	0    1    1    0
@@
 P 2300 4400
 F 0 "R3" V 2041 4400 50  0000 C CNN
-F 1 "7.87k" V 2132 4400 50  0000 C CNN
-F 2 "Resistors_SMD:R_0603" V 2204 4400 25  0000 C CNN
+F 1 "30.1" V 2132 4400 50  0000 C CNN
+F 2 "Resistor_SMD:R_0603_1608Metric" V 2204 4400 25  0000 C CNN
 F 3 "~" H 2300 4400 50  0001 C CNN
+F 4 "CRCW060330R1FKEA" H 0   0   50  0001 C CNN "part-num"
 	1    2300 4400
 	0    1    1    0
@@
 F 0 "R9" H 4230 3228 50  0000 R CNN
 F 1 "100k" H 4230 3319 50  0000 R CNN
-F 2 "Resistors_SMD:R_0603" H 4230 3391 25  0000 R CNN
+F 2 "Resistor_SMD:R_0603_1608Metric" H 4230 3391 25  0000 R CNN
 F 3 "~" H 4300 3300 50  0001 C CNN
+F 4 "CRCW0603100KFKEA" H 0   0   50  0001 C CNN "part-num"
 	1    4300 3300
 	-1   0    0    1
@@
 F 0 "R8" H 3630 3228 50  0000 R CNN
 F 1 "100k" H 3630 3319 50  0000 R CNN
-F 2 "Resistors_SMD:R_0603" H 3630 3391 25  0000 R CNN
+F 2 "Resistor_SMD:R_0603_1608Metric" H 3630 3391 25  0000 R CNN
 F 3 "~" H 3700 3300 50  0001 C CNN
+F 4 "CRCW0603100KFKEA" H 0   0   50  0001 C CNN "part-num"
 	1    3700 3300
 	-1   0    0    1
@@
 F 0 "R7" H 3030 3228 50  0000 R CNN
 F 1 "100k" H 3030 3319 50  0000 R CNN
-F 2 "Resistors_SMD:R_0603" H 3030 3391 25  0000 R CNN
+F 2 "Resistor_SMD:R_0603_1608Metric" H 3030 3391 25  0000 R CNN
 F 3 "~" H 3100 3300 50  0001 C CNN
+F 4 "CRCW0603100KFKEA" H 0   0   50  0001 C CNN "part-num"
 	1    3100 3300
 	-1   0    0    1
@@
 F 0 "R66" V 9891 2500 50  0000 C CNN
 F 1 "NF_30k" V 9982 2500 50  0000 C CNN
-F 2 "Resistors_SMD:R_0603" V 10054 2500 25  0000 C CNN
+F 2 "Resistor_SMD:R_0603_1608Metric" V 10054 2500 25  0000 C CNN
 F 3 "~" H 10150 2500 50  0001 C CNN
+F 4 "NF" H 0   0   50  0001 C CNN "part-num"
+F 5 "TRUE" H 0   0   50  0001 C CNN "DNP"
 	1    10150 2500
 	-1   0    0    1
@@
 F 2 "SC-70-5:SC-70-5" H 13100 2700 60  0001 C CNN
 F 3 "" H 13150 3050 60  0000 C CNN
+F 4 "SN74AUP1T17" H 0   0   50  0001 C CNN "part-num"
+F 5 "TRUE" H 0   0   50  0001 C CNN "DNP"
 	1    13100 3150
 	1    0    0    -1
@@
 F 0 "C97" H 12065 2472 50  0000 L CNN
 F 1 "NF_100n" H 12065 2381 50  0000 L CNN
-F 2 "Capacitors_SMD:C_0603" H 12065 2309 25  0000 L CNN
+F 2 "Capacitor_SMD:C_0603_1608Metric" H 12065 2309 25  0000 L CNN
 F 3 "~" H 11950 2400 50  0001 C CNN
+F 4 "NF" H 0   0   50  0001 C CNN "part-num"
+F 5 "TRUE" H 0   0   50  0001 C CNN "DNP"
 	1    11950 2400
 	1    0    0    -1
@@
 F 0 "R98" V 9991 3250 50  0000 C CNN
 F 1 "NF_30k" V 10082 3250 50  0000 C CNN
-F 2 "Resistors_SMD:R_0603" V 10154 3250 25  0000 C CNN
+F 2 "Resistor_SMD:R_0603_1608Metric" V 10154 3250 25  0000 C CNN
 F 3 "~" H 10250 3250 50  0001 C CNN
+F 4 "NF" H 0   0   50  0001 C CNN "part-num"
+F 5 "TRUE" H 0   0   50  0001 C CNN "DNP"
 	1    10250 3250
 	-1   0    0    1
@@
 F 0 "C95" H 10265 4972 50  0000 L CNN
 F 1 "NF_10n" H 10265 4881 50  0000 L CNN
-F 2 "Capacitors_SMD:C_0603" H 10265 4809 25  0000 L CNN
+F 2 "Capacitor_SMD:C_0603_1608Metric" H 10265 4809 25  0000 L CNN
 F 3 "~" H 10150 4900 50  0001 C CNN
+F 4 "NF" H 0   0   50  0001 C CNN "part-num"
+F 5 "TRUE" H 0   0   50  0001 C CNN "DNP"
 	1    10150 4900
 	1    0    0    -1
@@
 F 0 "C98" H 12215 4972 50  0000 L CNN
 F 1 "NF_10n" H 12215 4881 50  0000 L CNN
-F 2 "Capacitors_SMD:C_0603" H 12215 4809 25  0000 L CNN
+F 2 "Capacitor_SMD:C_0603_1608Metric" H 12215 4809 25  0000 L CNN
 F 3 "~" H 12100 4900 50  0001 C CNN
+F 4 "NF" H 0   0   50  0001 C CNN "part-num"
+F 5 "TRUE" H 0   0   50  0001 C CNN "DNP"
 	1    12100 4900
 	1    0    0    -1
@@
 F 0 "R67" V 9941 7000 50  0000 C CNN
 F 1 "NF_30k" V 10032 7000 50  0000 C CNN
-F 2 "Resistors_SMD:R_0603" V 10104 7000 25  0000 C CNN
+F 2 "Resistor_SMD:R_0603_1608Metric" V 10104 7000 25  0000 C CNN
 F 3 "~" H 10200 7000 50  0001 C CNN
+F 4 "NF" H 0   0   50  0001 C CNN "part-num"
+F 5 "TRUE" H 0   0   50  0001 C CNN "DNP"
 	1    10200 7000
 	-1   0    0    1
@@
 F 0 "TH1" H 10305 7822 50  0000 L CNN
 F 1 "NF_100k" H 10305 7731 50  0000 L CNN
-F 2 "Capacitors_SMD:C_0603" H 10305 7659 25  0000 L CNN
+F 2 "Capacitor_SMD:C_0603_1608Metric" H 10305 7659 25  0000 L CNN
 F 3 "~" H 10200 7750 50  0001 C CNN
+F 4 "NF" H 0   0   50  0001 C CNN "part-num"
+F 5 "TRUE" H 0   0   50  0001 C CNN "DNP"
 	1    10200 7750
 	1    0    0    -1
@@
 F 0 "R99" V 10841 7400 50  0000 C CNN
 F 1 "NF_0R" V 10932 7400 50  0000 C CNN
-F 2 "Resistors_SMD:R_0603" V 11004 7400 25  0000 C CNN
+F 2 "Resistor_SMD:R_0603_1608Metric" V 11004 7400 25  0000 C CNN
 F 3 "~" H 11100 7400 50  0001 C CNN
+F 4 "NF" H 0   0   50  0001 C CNN "part-num"
+F 5 "TRUE" H 0   0   50  0001 C CNN "DNP"
 	1    11100 7400
 	0    -1   -1   0
@@
 F 0 "C96" H 11565 7772 50  0000 L CNN
 F 1 "NF_10n" H 11565 7681 50  0000 L CNN
-F 2 "Capacitors_SMD:C_0603" H 11565 7609 25  0000 L CNN
+F 2 "Capacitor_SMD:C_0603_1608Metric" H 11565 7609 25  0000 L CNN
 F 3 "~" H 11450 7700 50  0001 C CNN
+F 4 "NF" H 0   0   50  0001 C CNN "part-num"
+F 5 "TRUE" H 0   0   50  0001 C CNN "DNP"
 	1    11450 7700
 	1    0    0    -1
