File: Design/Projector/DLP_Board/dlp_01/dlp_01_sch_brd/dmd.sch (KiCad schematic (older format))
At the start: 5 parts, among them U7 DLP3310AFQM

Commit message: Dump of uncommitted changes
Parts:
- C89, C90, C91, C92: footprint Capacitors_SMD:C_0805 -> Capacitor_SMD:C_0805_2012Metric; part-num (none) -> 0805ZC106KAT4A
- U7: part-num (none) -> DLP3310AFQM
Other:
- note added: "Mapping from p41 of DLPC3437 datasheet"
Changed lines of the file:
@@
 EESchema Schematic File Version 4
-EELAYER 30 0
+LIBS:dlp_01-cache
+EELAYER 26 0
 EELAYER END
 $Descr A3 16535 11693
@@
 F 2 "DLP3310:DLP3310" H 5400 1950 50  0001 C CNN
 F 3 "http://www.ti.com/lit/ds/symlink/dlp3310.pdf" H 5400 1950 50  0001 C CNN
+F 4 "DLP3310AFQM" H 0   0   50  0001 C CNN "part-num"
 	1    5400 1950
 	1    0    0    -1
@@
 F 2 "DLP3310:DLP3310" H 5400 7350 50  0001 C CNN
 F 3 "http://www.ti.com/lit/ds/symlink/dlp3310.pdf" H 5400 7350 50  0001 C CNN
+F 4 "DLP3310AFQM" H 0   0   50  0001 C CNN "part-num"
 	2    5400 7350
 	1    0    0    -1
@@
 F 2 "DLP3310:DLP3310" H 10650 4650 50  0001 C CNN
 F 3 "http://www.ti.com/lit/ds/symlink/dlp3310.pdf" H 10650 4650 50  0001 C CNN
+F 4 "DLP3310AFQM" H 0   0   50  0001 C CNN "part-num"
 	3    10650 4650
 	1    0    0    -1
@@
 F 0 "C92" H 10365 7472 50  0000 L CNN
 F 1 "10u" H 10365 7381 50  0000 L CNN
-F 2 "Capacitors_SMD:C_0805" H 10365 7309 25  0000 L CNN
+F 2 "Capacitor_SMD:C_0805_2012Metric" H 10365 7309 25  0000 L CNN
 F 3 "~" H 10250 7400 50  0001 C CNN
+F 4 "0805ZC106KAT4A" H 0   0   50  0001 C CNN "part-num"
 	1    10250 7400
 	1    0    0    -1
@@
 F 0 "C91" H 9765 7472 50  0000 L CNN
 F 1 "10u" H 9765 7381 50  0000 L CNN
-F 2 "Capacitors_SMD:C_0805" H 9765 7309 25  0000 L CNN
+F 2 "Capacitor_SMD:C_0805_2012Metric" H 9765 7309 25  0000 L CNN
 F 3 "~" H 9650 7400 50  0001 C CNN
+F 4 "0805ZC106KAT4A" H 0   0   50  0001 C CNN "part-num"
 	1    9650 7400
 	1    0    0    -1
@@
 F 0 "C90" H 9115 7472 50  0000 L CNN
 F 1 "10u" H 9115 7381 50  0000 L CNN
-F 2 "Capacitors_SMD:C_0805" H 9115 7309 25  0000 L CNN
+F 2 "Capacitor_SMD:C_0805_2012Metric" H 9115 7309 25  0000 L CNN
 F 3 "~" H 9000 7400 50  0001 C CNN
+F 4 "0805ZC106KAT4A" H 0   0   50  0001 C CNN "part-num"
 	1    9000 7400
 	1    0    0    -1
@@
 F 0 "C89" H 8515 7472 50  0000 L CNN
 F 1 "10u" H 8515 7381 50  0000 L CNN
-F 2 "Capacitors_SMD:C_0805" H 8515 7309 25  0000 L CNN
+F 2 "Capacitor_SMD:C_0805_2012Metric" H 8515 7309 25  0000 L CNN
 F 3 "~" H 8400 7400 50  0001 C CNN
+F 4 "0805ZC106KAT4A" H 0   0   50  0001 C CNN "part-num"
 	1    8400 7400
 	1    0    0    -1
@@
 Wire Wire Line
 	9350 7650 9650 7650
+Text Notes 2350 4550 0    50   ~ 0
+Mapping from p41 of DLPC3437 datasheet
 $EndSCHEMATC
